File: Wasabi.v1.1/Wasabi.v1.1.kicad_sch (KiCad schematic)
At the start: 16 parts, among them IC1 L298P, J1 Screw_Terminal_01x04, J2 Screw_Terminal_01x09, J3 Screw_Terminal_01x02, U1 Teensy4.1, U2 LF33ABV

Commit message: Update Wasabi.v1.1.kicad_sch
Parts:
- removed J2: Screw_Terminal_01x09, symbol Connector:Screw_Terminal_01x09
- removed J3: Screw_Terminal_01x02, symbol Connector:Screw_Terminal_01x02
- removed U2: LF33ABV, TO-220_STM, symbol 2024-01-19_00-29-09:LF33ABV
- added C3, C4, C5: C, symbol Device:C
- added J3: Screw_Terminal_01x08, symbol Connector:Screw_Terminal_01x08
- added J4: Screw_Terminal_01x07, symbol Connector:Screw_Terminal_01x07
- added J5: Conn_01x03_Pin, Connector:FanPinHeader_1x03_P2.54mm_Vertical, symbol Connector:Conn_01x03_Pin
- added J6: XT30PW-M, XT30PW-M:AMASS_XT30PW-M, symbol XT30PW-M:XT30PW-M
- added LED1, LED10, LED2, LED3, LED4, LED5, LED6, LED7, LED8, LED9: LTST-C191KRKT, LED_LTST-C191KRKT_LTO, symbol LED--:LTST-C191KRKT
- added R1, R10, R2, R3, R4, R5, R6, R7, R8, R9: R, symbol Device:R
- added U3: L78M05ABDT-TR, DPAK_STM, symbol L78M05ABDT-TR:L78M05ABDT-TR
Connections:
- net 7V is gone; now on net 7.4V Battery: C1.2, C2.2
- net +3.3V: now also U1.46 (3V3), J3.2 (Pin_2), J3.6 (Pin_6), J4.2 (Pin_2), J4.5 (Pin_5), J5.3 (Pin_3), R3.2
- net GND: now also C3.1, C4.1, C5.2, J3.1 (Pin_1), J3.5 (Pin_5), J4.1 (Pin_1), J4.4 (Pin_4), J5.2 (Pin_2), J6.N, LED1.1, LED10.1, LED2.1, LED3.1, LED4.1, LED5.1, LED6.1, LED7.1, LED8.1, LED9.1, U3.3 (GND)
- net Pin 17: now also J3.8 (Pin_8), R4.2
- net Pin 18: now also J3.7 (Pin_7), R5.2
- net Pin 19: now also J3.4 (Pin_4), R6.2
- net Pin 20: now also J3.3 (Pin_3), R7.2
- net Pin 21: now also J4.7 (Pin_7), R8.2
- net Pin 22: now also J4.6 (Pin_6), R9.2
- net Pin 23: now also J4.3 (Pin_3), R10.2
- net +5V: now reaches IC1.12 (VSS)
- net +5V: now also C3.2, C4.2, R2.2, U3.2 (OUTPUT)
- net 7.4V Battery: now reaches IC1.6 (VS)
- net 7.4V Battery: now also C5.1, J6.P, R1.2, U3.1 (INPUT)
- new net: LED10.2, R10.1
- new net: LED6.2, R6.1
- new net: LED5.2, R5.1
- new net: LED4.2, R4.1
- new net: LED9.2, R9.1
- new net: LED3.2, R3.1
- new net: LED7.2, R7.1
- new net: LED8.2, R8.1
- new net: LED1.2, R1.1
- new net: LED2.2, R2.1
- new net Signal: J5.1 (Pin_1)
- no-connect marks 0 -> 61
Other:
- note added: ".1µF"
- note added: ".33µF"
- note added: "100 Ohm"
- note added: "100nF"
- note added: "180 Ohm"
- note added: "50 Ohm"
- note added: "Blue for IR sensor"
- note added: "Green for Line Sensor"
- note added: "Orange for 5V"
- note added: "RED for 7.4V"
- note added: "Yellow for 3.3V"
