File: Wasabi.v1.1/wasabi(PCBlayout)/wasabi(PCBlayout).kicad_sch (KiCad schematic)
At the start: 49 parts, among them IC1 L298P, J1 Screw_Terminal_01x04, J2 Conn_01x03_Pin, J3 XT30PW-M, J4 Screw_Terminal_01x07, J5 Screw_Terminal_01x08, U1 HEF4104BT_653, U2 Teensy4.1, U3 HEF4104BT_653, U4 1101M2S3CQE2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

Commit message: Starting pcb layout
Parts:
- U2: footprint Wasabi(Footprints):TEENSY41(footprint) -> Wasabi(Footprints):Teensy41 (footprint NEW)
Connections:
- net +3.3V: now also U2.15 (3V3)
- net +5V: now also U2.48 (VIN)
- net GND: now also U2.34 (GND), U2.47 (GND)
- no-connect marks 70 -> 66
Changed lines of the file:
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@@
   )
   (no_connect (at 102.87 120.65))
-  (no_connect (at 102.87 83.82))
   (no_connect (at 102.87 76.2))
   (no_connect (at 46.99 93.98))
@@
   (no_connect (at 58.42 264.16))
   (no_connect (at 46.99 128.27))
-  (no_connect (at 102.87 48.26))
   (no_connect (at 217.17 261.62))
   (no_connect (at 102.87 73.66))
   (no_connect (at 67.31 135.89))
   (no_connect (at 46.99 71.12))
-  (no_connect (at 102.87 50.8))
   (no_connect (at 217.17 259.08))
-  (no_connect (at 46.99 83.82))
   (no_connect (at 46.99 114.3))
   (wire (pts (xy 45.085 165.1) (xy 62.865 165.1))
@@
     (effects (font (size 1.27 1.27)) (justify left bottom))
   )
-  (text "Input Pins \nfor Sensors" (at 104.775 48.26 0)
+  (text "Input Pins \nfor Sensors" (at 114.3 52.07 0)
     (effects (font (size 1.27 1.27)) (justify left bottom))
   )
@@
       (effects (font (size 1.27 1.27)))
     )
-    (property "Footprint" "Wasabi(Footprints):TEENSY41(footprint)" (at 64.77 92.71 0)
+    (property "Footprint" "Wasabi(Footprints):Teensy41 (footprint NEW)" (at 64.77 92.71 0)
       (effects (font (size 1.27 1.27)) hide)
     )
@@
     )
   )
+  (symbol (lib_id "power:+3.3V") (at 46.99 83.82 90) (unit 1)
+    (in_bom yes) (on_board yes) (dnp no) (fields_autoplaced)
+    (property "Reference" "#PWR042" (at 50.8 83.82 0)
+      (effects (font (size 1.27 1.27)) hide)
+    )
+    (property "Value" "+3.3V" (at 43.18 83.82 90)
+      (effects (font (size 1.27 1.27)) (justify left))
+    )
+    (property "Footprint" "" (at 46.99 83.82 0)
+      (effects (font (size 1.27 1.27)) hide)
+    )
+    (property "Datasheet" "" (at 46.99 83.82 0)
+      (effects (font (size 1.27 1.27)) hide)
+    )
+    (pin "1")
+    (instances
+      (project "wasabi(PCBlayout)"
+        (path "/2233659d-bbf8-40ca-afc8-264af30c67f0"
+          (reference "#PWR042") (unit 1)
+        )
+      )
+    )
+  )
   (symbol (lib_id "Device:R") (at 180.34 158.75 270) (unit 1)
     (in_bom yes) (on_board yes) (dnp no) (fields_autoplaced)
@@
     )
   )
+  (symbol (lib_id "power:GND") (at 102.87 83.82 90) (unit 1)
+    (in_bom yes) (on_board yes) (dnp no) (fields_autoplaced)
+    (property "Reference" "#PWR043" (at 109.22 83.82 0)
+      (effects (font (size 1.27 1.27)) hide)
+    )
+    (property "Value" "GND" (at 106.68 83.82 90)
+      (effects (font (size 1.27 1.27)) (justify right))
+    )
+    (property "Footprint" "" (at 102.87 83.82 0)
+      (effects (font (size 1.27 1.27)) hide)
+    )
+    (property "Datasheet" "" (at 102.87 83.82 0)
+      (effects (font (size 1.27 1.27)) hide)
+    )
+    (pin "1")
+    (instances
+      (project "wasabi(PCBlayout)"
+        (path "/2233659d-bbf8-40ca-afc8-264af30c67f0"
+          (reference "#PWR043") (unit 1)
+        )
+      )
+    )
+  )
   (symbol (lib_id "Device:C") (at 89.535 204.47 90) (unit 1)
     (in_bom yes) (on_board yes) (dnp no) (fields_autoplaced)
@@
     )
   )
+  (symbol (lib_id "power:+5V") (at 102.87 48.26 270) (mirror x) (unit 1)
+    (in_bom yes) (on_board yes) (dnp no) (fields_autoplaced)
+    (property "Reference" "#PWR045" (at 99.06 48.26 0)
+      (effects (font (size 1.27 1.27)) hide)
+    )
+    (property "Value" "+5V" (at 106.68 48.26 90)
+      (effects (font (size 1.27 1.27)) (justify left))
+    )
+    (property "Footprint" "" (at 102.87 48.26 0)
+      (effects (font (size 1.27 1.27)) hide)
+    )
+    (property "Datasheet" "" (at 102.87 48.26 0)
+      (effects (font (size 1.27 1.27)) hide)
+    )
+    (pin "1")
+    (instances
+      (project "wasabi(PCBlayout)"
+        (path "/2233659d-bbf8-40ca-afc8-264af30c67f0"
+          (reference "#PWR045") (unit 1)
+        )
+      )
+    )
+  )
   (symbol (lib_id "power:GND") (at 102.235 165.1 90) (unit 1)
     (in_bom yes) (on_board yes) (dnp no) (fields_autoplaced)
@@
         )
       )
+    )
+  )
+  (symbol (lib_id "power:GND") (at 102.87 50.8 90) (unit 1)
+    (in_bom yes) (on_board yes) (dnp no) (fields_autoplaced)
+    (property "Reference" "#PWR044" (at 109.22 50.8 0)
+      (effects (font (size 1.27 1.27)) hide)
+    )
+    (property "Value" "GND" (at 106.68 50.8 90)
+      (effects (font (size 1.27 1.27)) (justify right))
+    )
+    (property "Footprint" "" (at 102.87 50.8 0)
+      (effects (font (size 1.27 1.27)) hide)
+    )
+    (property "Datasheet" "" (at 102.87 50.8 0)
+      (effects (font (size 1.27 1.27)) hide)
+    )
+    (pin "1")
+    (instances
+      (project "wasabi(PCBlayout)"
+        (path "/2233659d-bbf8-40ca-afc8-264af30c67f0"
+          (reference "#PWR044") (unit 1)
+        )
+      )

Commit message: 02/07/24
Parts:
- C1: footprint Wasabi(Footprints):AMASS_XT30PW-M(footprint) -> Capacitor_SMD:C_0402_1005Metric_Pad0.74x0.62mm_HandSolder
Connections:
- net Signal is gone; now on net Signal Start Module: J2.1 (Pin_1)
- net Signal Start Module: now reaches U2.38 (16_A2_RX4_SCL1)
- no-connect marks 66 -> 65
Other:
- moved on the sheet: C1
Changed lines of the file:
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@@
   (no_connect (at 46.99 128.27))
   (no_connect (at 217.17 261.62))
-  (no_connect (at 102.87 73.66))
   (no_connect (at 67.31 135.89))
   (no_connect (at 46.99 71.12))
@@
     (stroke (width 0) (type default))
   )
+  (wire (pts (xy 86.36 187.96) (xy 85.725 187.96))
+    (stroke (width 0) (type default))
+  )
   (wire (pts (xy 184.785 39.37) (xy 196.215 39.37))
     (stroke (width 0) (type default))
@@
     (stroke (width 0) (type default))
   )
-  (wire (pts (xy 93.345 187.96) (xy 95.885 187.96))
+  (wire (pts (xy 93.98 187.96) (xy 95.885 187.96))
     (stroke (width 0) (type default))
   )
@@
     )
   )
-  (global_label "Signal" (shape input) (at 145.415 188.595 0) (fields_autoplaced)
-    (effects (font (size 1.27 1.27)) (justify left))
-    (property "Intersheetrefs" "${INTERSHEET_REFS}" (at 154.3267 188.595 0)
+  (global_label "Signal Start Module" (shape input) (at 145.415 188.595 0) (fields_autoplaced)
+    (effects (font (size 1.27 1.27)) (justify left))
+    (property "Intersheetrefs" "${INTERSHEET_REFS}" (at 167.5102 188.595 0)
       (effects (font (size 1.27 1.27)) (justify left) hide)
     )
@@
     (property "Intersheetrefs" "${INTERSHEET_REFS}" (at 16.7303 66.04 0)
       (effects (font (size 1.27 1.27)) (justify right) hide)
+    )
+  )
+  (global_label "Signal Start Module" (shape input) (at 102.87 73.66 0) (fields_autoplaced)
+    (effects (font (size 1.27 1.27)) (justify left))
+    (property "Intersheetrefs" "${INTERSHEET_REFS}" (at 124.9652 73.66 0)
+      (effects (font (size 1.27 1.27)) (justify left) hide)
     )
   )
@@
     )
   )
-  (symbol (lib_id "Device:C") (at 89.535 187.96 90) (unit 1)
-    (in_bom yes) (on_board yes) (dnp no) (fields_autoplaced)
-    (property "Reference" "C1" (at 89.535 180.34 90)
+  (symbol (lib_id "Device:C") (at 90.17 187.96 90) (unit 1)
+    (in_bom yes) (on_board yes) (dnp no) (fields_autoplaced)
+    (property "Reference" "C1" (at 90.17 180.34 90)
       (effects (font (size 1.27 1.27)))
     )
-    (property "Value" "C" (at 89.535 182.88 90)
+    (property "Value" "C" (at 90.17 182.88 90)
       (effects (font (size 1.27 1.27)))
     )
-    (property "Footprint" "Wasabi(Footprints):AMASS_XT30PW-M(footprint)" (at 93.345 186.9948 0)
-      (effects (font (size 1.27 1.27)) hide)
-    )
-    (property "Datasheet" "~" (at 89.535 187.96 0)
-      (effects (font (size 1.27 1.27)) hide)
-    )
+    (property "Footprint" "Capacitor_SMD:C_0402_1005Metric_Pad0.74x0.62mm_HandSolder" (at 93.98 186.9948 0)
+      (effects (font (size 1.27 1.27)) hide)
+    )
+    (property "Datasheet" "~" (at 90.17 187.96 0)
+      (effects (font (size 1.27 1.27)) hide)
+    )

Commit message: 02/12/24
Parts:
- added H1, H2: MountingHole, MountingHole:MountingHole_2.2mm_M2_DIN965, symbol Mechanical:MountingHole
Other:
- note added: "Mounting Holes"
Changed lines of the file:
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@@
     (effects (font (size 2.5 2.5)) (justify left bottom))
+  )
+  (text "Mounting Holes" (at 255.27 229.87 0)
+    (effects (font (size 6 6)) (justify left bottom))
   )
   (text "100nF" (at 92.075 186.69 0)
@@
     )
   )
+  (symbol (lib_id "Mechanical:MountingHole") (at 269.24 236.22 0) (unit 1)
+    (in_bom yes) (on_board yes) (dnp no) (fields_autoplaced)
+    (property "Reference" "H1" (at 271.78 234.95 0)
+      (effects (font (size 1.27 1.27)) (justify left))
+    )
+    (property "Value" "MountingHole" (at 271.78 237.49 0)
+      (effects (font (size 1.27 1.27)) (justify left))
+    )
+    (property "Footprint" "MountingHole:MountingHole_2.2mm_M2_DIN965" (at 269.24 236.22 0)
+      (effects (font (size 1.27 1.27)) hide)
+    )
+    (property "Datasheet" "~" (at 269.24 236.22 0)
+      (effects (font (size 1.27 1.27)) hide)
+    )
+    (instances
+      (project "wasabi(PCBlayout)"
+        (path "/2233659d-bbf8-40ca-afc8-264af30c67f0"
+          (reference "H1") (unit 1)
+        )
+      )
+    )
+  )
   (symbol (lib_id "Diode:RF01VM2S") (at 90.805 176.53 0) (unit 1)
     (in_bom yes) (on_board yes) (dnp no) (fields_autoplaced)
@@
         )
       )
+    )
+  )
+  (symbol (lib_id "Mechanical:MountingHole") (at 297.18 236.22 0) (unit 1)
+    (in_bom yes) (on_board yes) (dnp no) (fields_autoplaced)
+    (property "Reference" "H2" (at 299.72 234.95 0)
+      (effects (font (size 1.27 1.27)) (justify left))
+    )
+    (property "Value" "MountingHole" (at 299.72 237.49 0)
+      (effects (font (size 1.27 1.27)) (justify left))
+    )
+    (property "Footprint" "MountingHole:MountingHole_2.2mm_M2_DIN965" (at 297.18 236.22 0)
+      (effects (font (size 1.27 1.27)) hide)
+    )
+    (property "Datasheet" "~" (at 297.18 236.22 0)
+      (effects (font (size 1.27 1.27)) hide)
+    )
+    (instances
+      (project "wasabi(PCBlayout)"
+        (path "/2233659d-bbf8-40ca-afc8-264af30c67f0"
+          (reference "H2") (unit 1)
+        )
+      )

Commit message: final version (hopefully)
Connections:
- net GND: now also IC1.21 (EP)
- no-connect marks 65 -> 64
Changed lines of the file:
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@@
   (no_connect (at 217.17 266.7))
   (no_connect (at 260.35 43.18))
-  (no_connect (at 280.67 76.2))
   (no_connect (at 46.99 120.65))
   (no_connect (at 109.22 266.7))
@@
         )
       )
+    )
+  )
+  (symbol (lib_id "power:GND") (at 280.67 76.2 0) (unit 1)
+    (in_bom yes) (on_board yes) (dnp no) (fields_autoplaced)
+    (property "Reference" "#PWR046" (at 280.67 82.55 0)
+      (effects (font (size 1.27 1.27)) hide)
+    )
+    (property "Value" "GND" (at 280.67 81.28 0)
+      (effects (font (size 1.27 1.27)))
+    )
+    (property "Footprint" "" (at 280.67 76.2 0)
+      (effects (font (size 1.27 1.27)) hide)
+    )
+    (property "Datasheet" "" (at 280.67 76.2 0)
+      (effects (font (size 1.27 1.27)) hide)
+    )
+    (pin "1")
+    (instances
+      (project "wasabi(PCBlayout)"
+        (path "/2233659d-bbf8-40ca-afc8-264af30c67f0"
+          (reference "#PWR046") (unit 1)
+        )
+      )
