File: Wasabi.v1.1/wasabi(PCBlayout)/wasabi(PCBlayout).kicad_pcb (KiCad board)
At the start: 2 copper layers, 49 parts, among them IC1 L298P, J1 Screw_Terminal_01x04, J2 Conn_01x03_Pin, J3 XT30PW-M, J4 Screw_Terminal_01x07, J5 Screw_Terminal_01x08, U1 HEF4104BT_653, U2 Teensy4.1, U3 HEF4104BT_653, U4 1101M2S3CQE2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

Commit message: Starting pcb layout
Parts:
- removed C1: C, Wasabi(Footprints):AMASS_XT30PW-M(footprint)
- U2: footprint Wasabi(Footprints):TEENSY41(footprint) -> Wasabi(Footprints):Teensy41 (footprint NEW)
- moved D1 195.4 mm to (166.5, 158.0), turned to -90 degrees
- moved D2 188.1 mm to (161.0, 156.5), turned to -90 degrees
- moved D3 181.8 mm to (155.5, 156.5), turned to -90 degrees
- moved D4 177.1 mm to (152.2, 156.5), turned to -90 degrees
- moved D5 165.7 mm to (136.0, 159.5), turned to 90 degrees
- moved J1 160.6 mm to (140.0, 178.0), turned to 180 degrees
- moved D6 159.2 mm to (130.0, 159.4), turned to 90 degrees
- moved R9 157.9 mm to (182.5, 39.0), turned to 90 degrees
- moved D7 152.7 mm to (124.0, 159.4), turned to 90 degrees
- moved R4 147.8 mm to (174.0, 34.9), turned to 90 degrees
- moved D8 146.4 mm to (118.0, 159.4), turned to 90 degrees
- moved R6 141.6 mm to (165.0, 34.9), turned to 90 degrees
- moved R3 134.8 mm to (161.0, 35.0), turned to 90 degrees
- moved R7 130.5 mm to (151.5, 35.5), turned to 90 degrees
- moved R10 130.4 mm to (148.5, 35.5), turned to 90 degrees
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Connections:
- U2 pad 15: unconnected-(U2-3V3-Pad15) -> +3.3V
- U2 pad 34: unconnected-(U2-GND-Pad34) -> GND
- U2 pad 47: unconnected-(U2-GND-Pad47) -> GND
- U2 pad 48: unconnected-(U2-VIN-Pad48) -> +5V

Commit message: 02/07/24
Parts:
- added C1: C, Capacitor_SMD:C_0402_1005Metric_Pad0.74x0.62mm_HandSolder, F.Cu at (128.5, 196.1)
- moved J2 152.6 mm to (183.8, 53.1)
- moved C7 141.7 mm to (169.4, 48.1)
- moved C6 131.1 mm to (158.8, 48.6)
- moved C9 118.5 mm to (158.5, 128.1), turned to 90 degrees
- moved C4 117.7 mm to (144.8, 48.6)
- moved C3 110.4 mm to (137.3, 48.1)
- moved LED2 106.3 mm to (73.0, 137.3), turned to 90 degrees
- moved C5 106.2 mm to (77.5, 121.9), turned to 90 degrees
- moved U4 103.4 mm to (83.0, 142.2), turned to 180 degrees
- moved F1 98.0 mm to (83.0, 148.6), turned to 90 degrees
- moved U5 84.0 mm to (85.5, 119.5)
- moved LED8 82.7 mm to (96.7, 119.5)
- moved C2 59.2 mm to (121.0, 195.0), turned to -90 degrees
- moved R2 56.8 mm to (75.0, 132.5)
- moved LED4 54.6 mm to (170.4, 43.1)
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Connections:
- J2 pad 1: Signal -> Signal Start Module
- U2 pad 38: unconnected-(U2-16_A2_RX4_SCL1-Pad38) -> Signal Start Module
Routing:
- net 7.4V Battery(Pre Switch): track 0.00 -> 11.6 mm
- net 7.4V Battery(Pre fuse): track 0.00 -> 7.12 mm
- net 7.4V Battery: track 0.00 -> 5.95 mm

Commit message: 02/08/24
Parts:
- J3: moved to B.Cu
- moved J3 161.5 mm to (202.0, 61.3), turned to 0 degrees
- moved LED2 148.4 mm to (207.7, 74.9), turned to -90 degrees
- moved F1 143.4 mm to (205.2, 73.5), turned to -90 degrees
- moved R2 141.9 mm to (206.6, 79.7), turned to 180 degrees
- moved U4 136.2 mm to (199.0, 70.8), turned to 0 degrees
- moved C5 131.5 mm to (204.6, 88.1), turned to -90 degrees
- moved C1 124.8 mm to (185.5, 85.0), turned to 0 degrees
- moved C2 122.4 mm to (185.5, 91.0), turned to 0 degrees
- moved U5 117.3 mm to (199.2, 90.6), turned to 180 degrees
- moved D1 116.9 mm to (181.4, 83.5), turned to 180 degrees
- moved D4 116.7 mm to (181.4, 92.5), turned to 180 degrees
- moved D2 115.9 mm to (181.4, 86.5), turned to 180 degrees
- moved D3 115.5 mm to (181.4, 89.5), turned to 180 degrees
- moved C8 107.1 mm to (193.0, 85.5), turned to 90 degrees
- moved R8 100.7 mm to (189.9, 84.9), turned to 0 degrees
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Routing:
- net +5V: track 0.00 -> 41.8 mm, vias 0 -> 2
- net Pin 4 (3.3v sig MD): track 0.00 -> 18.9 mm
- net Pin 3 (3.3v sig MD): track 0.00 -> 17.4 mm
- net 7.4V Battery(Pre Switch): track 11.6 -> 0.00 mm
- net OUT 4: track 0.00 -> 10.9 mm
- net OUT 3: track 0.00 -> 10.6 mm
- net OUT 1: track 0.00 -> 10.5 mm
- net OUT 2: track 0.00 -> 10.1 mm
- net GND: track 0.00 -> 9.08 mm
- net Pin 5 (PWM for Speed 3.3v): track 0.00 -> 8.13 mm
- net 7.4V Battery(Pre fuse): track 7.12 -> 0.00 mm
- net Pin 6 (PWM for Speed 3.3v): track 0.00 -> 7.03 mm
- net Pin 1 (3.3v sig MD): track 0.00 -> 6.54 mm
- net Pin 2 (3.3v sig MD): track 0.00 -> 6.01 mm
- net 7.4V Battery: track 5.95 -> 0.30 mm
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
Commit message: 02/11/24
Parts:
- turned R1 to 90 degrees
Routing:
- net +3.3V: track 0.00 -> 153.8 mm
- net +5V: track 41.8 -> 178.8 mm, vias 2 -> 4
- net 7.4V Battery: track 0.30 -> 79.4 mm
- net Pin 4 (5v to MD): track 0.00 -> 63.6 mm
- net Pin 3 (5v to MD): track 0.00 -> 56.9 mm
- net Pin 6 (PWM for Speed 5v): track 0.00 -> 41.6 mm, vias 0 -> 2
- net Pin 2 (5v to MD): track 0.00 -> 40.3 mm
- net Pin 1 (5v to MD): track 0.00 -> 37.8 mm
- net Pin 5 (PWM for Speed 5v): track 0.00 -> 34.6 mm, vias 0 -> 2
- net Signal Start Module: track 0.00 -> 28.0 mm
- net Signal IR 1 (3.3v): track 0.00 -> 27.0 mm
- net Signal IR 2 (3.3v): track 0.00 -> 26.8 mm
- net 7.4V Battery(Pre fuse): track 0.00 -> 23.7 mm
- net Signal IR 3 (3.3v): track 0.00 -> 21.8 mm
- net Signal IR 4 (3.3v): track 0.00 -> 21.6 mm
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- added copper zone on F.Cu, net GND

Commit message: 02/12/24
Parts:
- added H1: MountingHole, MountingHole:MountingHole_2.2mm_M2_DIN965, F.Cu at (174.5, 97.5)
- added H2: MountingHole, MountingHole:MountingHole_2.2mm_M2_DIN965, F.Cu at (164.5, 97.5)
Routing:
- net GND: track 0.28 -> 2.90 mm, vias 0 -> 8
- added copper zone on B.Cu, net GND
Other:
- board outline added: 83 x 57.5 mm
Changed lines of the file:
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@@
   (setup
     (pad_to_mask_clearance 0)
+    (aux_axis_origin 127 103)
     (pcbplotparams
       (layerselection 0x00010fc_ffffffff)
@@
     )
   )
+  (footprint "MountingHole:MountingHole_2.2mm_M2_DIN965" (layer "F.Cu")
+    (at 164.5 97.5)
+    (descr "Mounting Hole 2.2mm, no annular, M2, DIN965")
+    (tags "mounting hole 2.2mm no annular m2 din965")
+    (property "Sheetfile" "wasabi(PCBlayout).kicad_sch")
+    (property "Sheetname" "")
+    (property "ki_description" "Mounting Hole without connection")
+    (property "ki_keywords" "mounting hole")
+    (attr exclude_from_pos_files)
+    (fp_text reference "H2" (at 0 -2.9) (layer "F.SilkS")
+        (effects (font (size 1 1) (thickness 0.15)))
+    )
+    (fp_text value "MountingHole" (at 0 2.9) (layer "F.Fab")
+        (effects (font (size 1 1) (thickness 0.15)))
+    )
+    (fp_text user "${REFERENCE}" (at 0 0) (layer "F.Fab")
+        (effects (font (size 1 1) (thickness 0.15)))
+    )
+    (fp_circle (center 0 0) (end 1.9 0)
+      (stroke (width 0.15) (type solid)) (fill none) (layer "Cmts.User"))
+    (fp_circle (center 0 0) (end 2.15 0)
+      (stroke (width 0.05) (type solid)) (fill none) (layer "F.CrtYd"))
+    (pad "" np_thru_hole circle (at 0 0) (size 2.2 2.2) (drill 2.2) (layers "*.Cu" "*.Mask"))
+  )
   (footprint "Wasabi(Footprints):LED_LTST-C191KRKT_LTO(footprint)" (layer "F.Cu")
     (at 160 47.5)
@@
     )
   )
+  (footprint "MountingHole:MountingHole_2.2mm_M2_DIN965" (layer "F.Cu")
+    (at 174.5 97.5)
+    (descr "Mounting Hole 2.2mm, no annular, M2, DIN965")
+    (tags "mounting hole 2.2mm no annular m2 din965")
+    (property "Sheetfile" "wasabi(PCBlayout).kicad_sch")
+    (property "Sheetname" "")
+    (property "ki_description" "Mounting Hole without connection")
+    (property "ki_keywords" "mounting hole")
+    (attr exclude_from_pos_files)
+    (fp_text reference "H1" (at 0 -2.9) (layer "F.SilkS")
+        (effects (font (size 1 1) (thickness 0.15)))
+    )
+    (fp_text value "MountingHole" (at 0 2.9) (layer "F.Fab")
+        (effects (font (size 1 1) (thickness 0.15)))
+    )
+    (fp_text user "${REFERENCE}" (at 0 0) (layer "F.Fab")
+        (effects (font (size 1 1) (thickness 0.15)))
+    )
+    (fp_circle (center 0 0) (end 1.9 0)
+      (stroke (width 0.15) (type solid)) (fill none) (layer "Cmts.User"))
+    (fp_circle (center 0 0) (end 2.15 0)
+      (stroke (width 0.05) (type solid)) (fill none) (layer "F.CrtYd"))
+    (pad "" np_thru_hole circle (at 0 0) (size 2.2 2.2) (drill 2.2) (layers "*.Cu" "*.Mask"))
+  )
   (footprint "Capacitor_SMD:C_0402_1005Metric_Pad0.74x0.62mm_HandSolder" (layer "F.Cu")
     (at 158.7072 52)
@@
       (solder_mask_margin 0.102))
   )
+  (gr_poly
+    (pts
+      (xy 127.5 44.5)
+      (xy 210.5 44.5)
+      (xy 210 102)
+      (xy 127.5 101.5)
+    )
+    (stroke (width 0.1) (type solid)) (fill none) (layer "Edge.Cuts"))
   (segment (start 182.85 86.5) (end 183.45 86.5) (width 0.25) (layer "F.Cu") (net 1))
   (segment (start 184.35 85) (end 182.85 83.5) (width 0.25) (layer "F.Cu") (net 1))
@@
   (segment (start 175.87 92.5) (end 180.05 92.5) (width 0.25) (layer "F.Cu") (net 6))
   (segment (start 174.03 92.5) (end 174.95 91.58) (width 0.25) (layer "F.Cu") (net 6))
+  (segment (start 169.5 48) (end 169.5 47.5) (width 0.25) (layer "F.Cu") (net 7))
   (segment (start 167.15 89.6) (end 167.05 89.5) (width 0.25) (layer "F.Cu") (net 7))
   (segment (start 167.05 86.6) (end 167.15 86.5) (width 0.25) (layer "F.Cu") (net 7))
+  (segment (start 171 49.5) (end 169.5 48) (width 0.25) (layer "F.Cu") (net 7))
+  (via (at 138.5 85.5) (size 0.8) (drill 0.4) (layers "F.Cu" "B.Cu") (free) (net 7))
+  (via (at 167.5 50) (size 0.8) (drill 0.4) (layers "F.Cu" "B.Cu") (free) (net 7))
+  (via (at 174.5 51) (size 0.8) (drill 0.4) (layers "F.Cu" "B.Cu") (free) (net 7))
+  (via (at 143 95) (size 0.8) (drill 0.4) (layers "F.Cu" "B.Cu") (free) (net 7))
+  (via (at 181.5 97) (size 0.8) (drill 0.4) (layers "F.Cu" "B.Cu") (free) (net 7))
+  (via (at 155 52) (size 0.8) (drill 0.4) (layers "F.Cu" "B.Cu") (free) (net 7))
+  (via (at 160.5 50.5) (size 0.8) (drill 0.4) (layers "F.Cu" "B.Cu") (free) (net 7))
+  (via (at 171 49.5) (size 0.8) (drill 0.4) (layers "F.Cu" "B.Cu") (free) (net 7))
   (segment (start 183.8 54) (end 181.5 54) (width 0.25) (layer "F.Cu") (net 8))
   (segment (start 181.5 54) (end 173.5 62) (width 0.25) (layer "F.Cu") (net 8))
@@
         (xy 123 42.5)
         (xy 212.5 42.5)
-        (xy 212.5 102)
-        (xy 122 101.5)
+        (xy 212.5 102.5)
+        (xy 122 102)
+      )
+    )
+  )
+  (zone (net 7) (net_name "GND") (layer "B.Cu") (hatch edge 0.5)
+    (priority 1)
+    (connect_pads (clearance 0.5))
+    (min_thickness 0.25) (filled_areas_thickness no)
+    (fill yes (thermal_gap 0.5) (thermal_bridge_width 0.5))
+    (polygon
+      (pts
+        (xy 123 42.5)
+        (xy 212.5 42.5)
+        (xy 212.5 102.5)
+        (xy 122 102)
       )
     )

Commit message: 02/12/24 (1:23pm)
Routing:
- net GND: track 2.90 -> 64.0 mm, vias 8 -> 16
- net Pin 6 (PWM for Speed 5v): track 41.6 -> 38.2 mm
- net Pin 3 (5v to MD): track 56.9 -> 59.3 mm
- net Pin 5 (PWM for Speed 5v): track 34.6 -> 35.7 mm

Commit message: 4/2/24
Connections:
- IC1 pad 21: unconnected-(IC1-EP-Pad21) -> GND
Routing:
- net GND: track 64.0 -> 79.3 mm
